File: JCM800.kicad_pcb (KiCad board)
At the start: 2 copper layers, 258.5 x 77.3 mm, 104 parts, among them U1 ECC83, U2 ECC83, U3 ECC83, U4 EL84, U5 EL84

Commit message: Preparing initial release
Parts:
- moved R31 3.09 mm to (180.3, 118.4)
- moved R32 3.09 mm to (186.9, 118.4)
- moved R33 3.09 mm to (186.9, 92.5)
- moved R36 3.09 mm to (180.3, 92.5)
- moved C10 3.05 mm to (255.0, 63.0)
- moved C15 3.05 mm to (125.2, 111.8)
- moved C3 3.05 mm to (63.0, 95.0)
- moved A1 3.05 mm to (274.1, 65.0)
- moved AC1 3.05 mm to (240.1, 58.4)
- moved BASS1 3.05 mm to (171.0, 127.3)
- moved C13 3.05 mm to (145.5, 104.3)
- moved C14 3.05 mm to (115.1, 111.8)
- moved C16 3.05 mm to (136.7, 96.0)
- moved C17 3.05 mm to (137.2, 73.0)
- moved C19 3.05 mm to (168.5, 116.1)
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Routing:
- net Net-(C19-Pad2): track 73.9 -> 76.4 mm
- net Net-(R32-Pad1): track 41.7 -> 42.3 mm

Commit message: Logo
Parts:
- added G***: LOGO, toad-logo:toad-big, F.Cu at (100.3, 109.0)
Other:
- board text added: "dazz"
- board text removed: "dazz's"

Commit message: Tweaks
Parts:
- moved G*** 0.25 mm to (100.3, 108.7)
Connections:
- net Net-(C20-Pad1) renamed /K

Commit message: Fixed bias
Parts:
- removed C20: 47u, Capacitor_THT:CP_Radial_D10.0mm_P3.50mm
- removed G***: LOGO, toad-logo:toad-big
- removed R22, R23: 100R, Resistor_THT:R_Axial_DIN0207_L6.3mm_D2.5mm_P10.16mm_Horizontal
- removed Rbias1: 180R/5W, Resistor_THT:R_Axial_DIN0922_L20.0mm_D9.0mm_P7.62mm_Vertical
- added BIAS1: B1M, Potentiometer_THT:Potentiometer_Bourns_3296W_Vertical, F.Cu at (209.2, 56.4)
- added BIAS2: B1M, Potentiometer_THT:Potentiometer_Bourns_3296W_Vertical, F.Cu at (209.2, 63.5)
- added C23: 47u, Capacitor_THT:CP_Radial_D6.3mm_P2.50mm, F.Cu at (176.0, 63.0)
- added C24: 47u, Capacitor_THT:CP_Radial_D6.3mm_P2.50mm, F.Cu at (190.0, 57.4)
- added D5: D, Diode_THT:D_A-405_P10.16mm_Horizontal, F.Cu at (175.3, 56.4)
- added GND8: GND, Connector_PinHeader_2.54mm:PinHeader_1x01_P2.54mm_Vertical, F.Cu at (132.3, 118.1)
- added LOGO1: LOGO, toad-logo:toad-big, F.Cu at (100.3, 108.6)
- added R39: 47K, Resistor_THT:R_Axial_DIN0207_L6.3mm_D2.5mm_P10.16mm_Horizontal, F.Cu at (182.9, 64.0)
- added R40: 47K, Resistor_THT:R_Axial_DIN0207_L6.3mm_D2.5mm_P10.16mm_Horizontal, F.Cu at (198.1, 65.0)
- added R41: 47K, Resistor_THT:R_Axial_DIN0207_L6.3mm_D2.5mm_P10.16mm_Horizontal, F.Cu at (220.1, 54.9)
- added R42: 47K, Resistor_THT:R_Axial_DIN0207_L6.3mm_D2.5mm_P10.16mm_Horizontal, F.Cu at (203.2, 65.0)
- moved GND5 143.0 mm to (80.3, 113.8)
- moved GND7 93.3 mm to (235.7, 118.4)
- moved R16 79.4 mm to (155.4, 113.3)
- moved H6 64.0 mm to (122.4, 57.4)
- moved GND9 40.7 mm to (149.9, 76.7)
- moved R31 39.6 mm to (214.9, 98.9), turned to 270 degrees
- moved R37 34.7 mm to (180.3, 118.4)
- moved H2 34.5 mm to (157.0, 57.4)
- moved GND6 27.6 mm to (235.7, 108.7)
- moved R30 5.72 mm to (208.5, 109.1)
- moved OUT1 3.48 mm to (144.6, 58.4)
- moved C19 3.05 mm to (171.6, 116.1)
- moved R28 3.05 mm to (163.1, 109.2)
- moved R29 3.05 mm to (173.2, 102.9)
- moved NFB2 2.54 mm to (274.1, 107.7)
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Connections:
- net /FIL2 renamed /FIL
- FIL1 pad 2: /FIL1 -> GNDS
- R30 pad 2: GNDS -> /BIAS1
- R31 pad 1: GNDS -> /BIAS2
- U1 pad 5: /FIL1 -> GNDS
- U2 pad 5: /FIL1 -> GNDS
- U3 pad 5: /FIL1 -> GNDS
- U4 pad 3: /K -> GND
- U5 pad 3: /K -> GND
- U5 pad 5: /FIL1 -> GNDS
Routing:
- net /FIL1: track 243.9 -> 0.00 mm, vias 3 -> 0
- net GNDS: track 0.00 -> 172.0 mm, vias 0 -> 2
- net /K: track 83.4 -> 0.00 mm
- net /D: track 203.3 -> 124.0 mm
- net /BIAS1: track 0.00 -> 75.0 mm, vias 0 -> 2
- net /BIAS2: track 0.00 -> 49.6 mm
- net Net-(BIAS1-Pad1): track 0.00 -> 44.3 mm
- net Net-(NFB1-Pad2): track 51.9 -> 88.7 mm
- net Net-(C19-Pad1): track 24.5 -> 54.7 mm
- net Net-(BIAS1-Pad3): track 0.00 -> 18.9 mm
- net /C: track 143.4 -> 161.7 mm
- net Net-(C23-Pad2): track 0.00 -> 13.4 mm
- net /B: track 104.0 -> 98.5 mm
- net /TO_PA: track 80.8 -> 77.5 mm, vias 1 -> 0
- net /4ohm: track 20.7 -> 23.3 mm
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Other:
- board text removed: "12.6V Heaters"

Commit message: Tweaks
Parts:
- moved GND5 147.1 mm to (227.1, 104.6)
- moved GND8 87.7 mm to (218.9, 104.6)
- moved R40 0.13 mm to (198.1, 65.2)
- moved R42 0.13 mm to (203.2, 65.2)
Connections:
- GND5 pad 1: GNDS -> GND
Routing:
- net GNDS: track 172.0 -> 0.55 mm, vias 2 -> 0
- net Net-(R2-Pad1): track 28.2 -> 21.6 mm
- net Net-(R20-Pad2): track 58.3 -> 62.9 mm
- net /FIL: track 182.2 -> 177.8 mm, vias 2 -> 4
- net Net-(BOOST1-Pad1): track 44.5 -> 41.1 mm
- net /C: track 161.7 -> 158.9 mm
- net Net-(NFB1-Pad2): track 88.7 -> 87.3 mm
- net Net-(C1-Pad1): track 38.9 -> 38.0 mm
- net /BIAS1: track 75.0 -> 75.8 mm
- net Net-(R17-Pad2): track 51.5 -> 52.0 mm, vias 1 -> 0

Commit message: Test points added. Trimmers moved further away from pentode.
Parts:
- removed BIAS1, BIAS2: B1M, Potentiometer_THT:Potentiometer_Bourns_3296W_Vertical
- added BIAS_U4: B1M, Potentiometer_THT:Potentiometer_Bourns_3296W_Vertical, F.Cu at (214.1, 56.1)
- added BIAS_U5: B1M, Potentiometer_THT:Potentiometer_Bourns_3296W_Vertical, F.Cu at (221.0, 56.1)
- added TC1: C, Connector_PinHeader_2.54mm:PinHeader_1x01_P2.54mm_Vertical, F.Cu at (274.4, 101.2)
- added TD1: D, Connector_PinHeader_2.54mm:PinHeader_1x01_P2.54mm_Vertical, F.Cu at (116.3, 57.3)
- added TE1: E, Connector_PinHeader_2.54mm:PinHeader_1x01_P2.54mm_Vertical, F.Cu at (45.8, 57.1)
- AB1: renamed from A1; value A -> AB
- C23, C24: value 47u -> 68u
- moved R41 11.8 mm to (208.3, 55.2)
- moved GND2 2.92 mm to (216.3, 69.3)
- moved GND4 0.60 mm to (228.1, 58.4)
- moved R40 0.25 mm to (198.1, 65.4)
- moved R42 0.25 mm to (203.2, 65.4)
Connections:
- AB1 pad 2: (no net) -> /B
Routing:
- net /B: track 98.5 -> 119.2 mm, vias 0 -> 1
- net /D: track 124.3 -> 143.1 mm
- net /BIAS2: track 49.6 -> 57.6 mm, vias 0 -> 2
- net /E: track 99.4 -> 103.7 mm
- net /A: track 91.6 -> 88.3 mm
- net /C: track 158.9 -> 161.6 mm
- net /BIAS1: track 75.8 -> 73.5 mm
- net Net-(BIAS_U4-Pad3): track 19.3 -> 20.2 mm
- net Net-(BIAS_U4-Pad1): track 44.3 -> 43.5 mm
Other:
- board text added: "12AX7#1"
- board text added: "12AX7#2"
- board text added: "INV"
- board text added: "PLATE"
- board text added: "SCREEN"
