File: JCM800.kicad_pcb (KiCad board)
At the start: 2 copper layers, 196 x 77.3 mm, 77 parts, among them U1 ECC83, U2 ECC83, U3 EL84

Commit message: Tweaks
Parts:
- moved C16 2.92 mm to (177.5, 59.8), turned to 0 degrees
- moved G*** 0.25 mm to (126.7, 110.0)
Routing:
- net /EL84-CATHODE: track 31.9 -> 33.9 mm
Other:
- board text added: "Single Ended"
- board text removed: "12AX7"
Changed lines of the file:
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@@
     (thickness 1.6)
     (drawings 11)
-    (tracks 329)
+    (tracks 325)
     (zones 0)
     (modules 77)
@@
   )
   (module toad-logo:toad-big (layer F.Cu)
-    (at 126.746 110.236)
+    (at 126.746 109.982)
     (fp_text reference G*** (at 0 0) (layer F.SilkS) hide
       (effects (font (size 1.524 1.524) (thickness 0.3)))
@@
     (descr "terminal block Metz Connect Type094_RT03502HBLU, 2 pins, pitch 5mm, size 10x8.3mm^2, drill diamater 1.3mm, pad diameter 2.6mm, see http://www.metz-connect.com/ru/system/files/productfiles/Data_sheet_310941_RT035xxHBLU_OFF-022742T.pdf, script-generated using https://github.com/pointhi/kicad-footprint-generator/scripts/TerminalBlock_MetzConnect")
     (tags "THT terminal block Metz Connect Type094_RT03502HBLU pitch 5mm size 10x8.3mm^2 drill 1.3mm pad 2.6mm")
-    (fp_text reference FIL1 (at 10.033 -3.048) (layer F.SilkS)
+    (fp_text reference FIL1 (at -4.699 1.905) (layer F.SilkS)
       (effects (font (size 1 1) (thickness 0.15)))
     )
@@
   )
   (module Capacitor_THT:CP_Radial_D8.0mm_P3.50mm (layer F.Cu)
-    (at 179.197 62.23 90)
+    (at 177.546 59.817)
     (descr "CP, Radial series, Radial, pin pitch=3.50mm, , diameter=8mm, Electrolytic Capacitor")
     (tags "CP Radial series Radial pin pitch 3.50mm  diameter 8mm Electrolytic Capacitor")
-    (fp_text reference C16 (at 6.858 -0.254 180) (layer F.SilkS)
+    (fp_text reference C16 (at 1.778 5.334) (layer F.SilkS)
       (effects (font (size 1 1) (thickness 0.15)))
     )
-    (fp_text value 22u (at 1.75 5.25 90) (layer F.Fab)
+    (fp_text value 22u (at 1.75 5.25) (layer F.Fab)
       (effects (font (size 1 1) (thickness 0.15)))
     )
@@
     (fp_line (start -2.659698 -2.315) (end -1.859698 -2.315) (layer F.SilkS) (width 0.12))
     (fp_line (start -2.259698 -2.715) (end -2.259698 -1.915) (layer F.SilkS) (width 0.12))
-    (fp_text user %R (at 1.75 0 90) (layer F.Fab)
+    (fp_text user %R (at 1.75 0) (layer F.Fab)
       (effects (font (size 1 1) (thickness 0.15)))
     )
-    (pad 1 thru_hole rect (at 0 0 90) (size 1.6 1.6) (drill 0.8) (layers *.Cu *.Mask)
+    (pad 1 thru_hole rect (at 0 0) (size 1.6 1.6) (drill 0.8) (layers *.Cu *.Mask)
       (net 37 /EL84-CATHODE))
-    (pad 2 thru_hole circle (at 3.5 0 90) (size 1.6 1.6) (drill 0.8) (layers *.Cu *.Mask)
+    (pad 2 thru_hole circle (at 3.5 0) (size 1.6 1.6) (drill 0.8) (layers *.Cu *.Mask)
       (net 6 GND))
     (model ${KISYS3DMOD}/Capacitor_THT.3dshapes/CP_Radial_D8.0mm_P3.50mm.wrl
@@
     (effects (font (size 1.5 1.5) (thickness 0.3)))
   )
-  (gr_text 6.3V (at 175.26 58.801) (layer F.SilkS)
+  (gr_text 6.3V (at 160.401 63.754) (layer F.SilkS)
     (effects (font (size 1 1) (thickness 0.15)))
   )
-  (gr_text 12AX7 (at 183.388 90.678) (layer F.SilkS)
+  (gr_text " Single \nEnded" (at 183.896 88.9) (layer F.SilkS)
     (effects (font (size 2.5 2.5) (thickness 0.3)))
   )
@@
     (effects (font (size 1 1) (thickness 0.15)))
   )
-  (gr_text v0.2 (at 144.272 80.772) (layer F.SilkS)
+  (gr_text v0.2 (at 144.272 80.01) (layer F.SilkS)
     (effects (font (size 3 3) (thickness 0.3)))
   )
@@
   (segment (start 52.832 98.044) (end 52.180868 97.424058) (width 0.5) (layer B.Cu) (net 4))
   (segment (start 56.134 101.346) (end 52.832 98.044) (width 0.5) (layer B.Cu) (net 4))
-  (segment (start 73.66 99.314) (end 71.628 101.346) (width 0.5) (layer B.Cu) (net 4))
+  (segment (start 73.66 99.314) (end 71.628 101.346) (width 0.5) (layer B.Cu) (net 4) (status 10))
   (segment (start 71.628 101.346) (end 56.134 101.346) (width 0.5) (layer B.Cu) (net 4))
-  (segment (start 52.180868 96.536132) (end 52.197 96.52) (width 0.5) (layer B.Cu) (net 4))
-  (segment (start 52.180868 97.424058) (end 52.180868 96.536132) (width 0.5) (layer B.Cu) (net 4))
+  (segment (start 52.180868 96.536132) (end 52.197 96.52) (width 0.5) (layer B.Cu) (net 4) (status 30))
+  (segment (start 52.180868 97.424058) (end 52.180868 96.536132) (width 0.5) (layer B.Cu) (net 4) (status 20))
   (segment (start 83.82 97.79) (end 83.82 90.043) (width 0.5) (layer F.Cu) (net 5))
   (segment (start 83.82 90.043) (end 82.296 88.519) (width 0.5) (layer F.Cu) (net 5))
@@
   (segment (start 114.427 105.316) (end 118.03 108.919) (width 0.5) (layer F.Cu) (net 9))
   (segment (start 114.427 105.283) (end 114.427 105.316) (width 0.5) (layer F.Cu) (net 9))
-  (segment (start 55.88 82.55) (end 59.25 80.166) (width 0.5) (layer F.Cu) (net 9))
+  (segment (start 55.88 82.55) (end 59.25 80.166) (width 0.5) (layer F.Cu) (net 9) (status 20))
   (segment (start 55.88 94.996) (end 55.88 82.55) (width 0.5) (layer F.Cu) (net 9))
   (segment (start 59.436 98.552) (end 55.88 94.996) (width 0.5) (layer F.Cu) (net 9))
@@
   (segment (start 82.804 104.14) (end 61.468 104.14) (width 0.5) (layer F.Cu) (net 9))
   (segment (start 111.76 104.19863) (end 110.43137 102.87) (width 0.5) (layer F.Cu) (net 9))
-  (segment (start 111.76 105.33) (end 111.76 104.19863) (width 0.5) (layer F.Cu) (net 9))
+  (segment (start 111.76 105.33) (end 111.76 104.19863) (width 0.5) (layer F.Cu) (net 9) (status 10))
   (segment (start 110.43137 102.87) (end 95.758 102.87) (width 0.5) (layer F.Cu) (net 9))
   (segment (start 95.758 102.87) (end 91.44 107.188) (width 0.5) (layer F.Cu) (net 9))
@@
   (segment (start 220.345 65.024) (end 218.145 65.024) (width 1) (layer F.Cu) (net 12) (status 10))
   (segment (start 216.027 66.421) (end 216.027 65.024) (width 1) (layer F.Cu) (net 12))
-  (segment (start 162.43999 56.12701) (end 213.868 56.12701) (width 1) (layer F.Cu) (net 12))
   (segment (start 160.782 61.722) (end 160.782 57.785) (width 1) (layer F.Cu) (net 12))
   (segment (start 160.782 57.785) (end 162.43999 56.12701) (width 1) (layer F.Cu) (net 12))
   (segment (start 216.027 58.166) (end 213.868 56.12701) (width 1) (layer F.Cu) (net 12))
   (segment (start 216.027 65.024) (end 216.027 58.166) (width 1) (layer F.Cu) (net 12))
+  (segment (start 162.43999 56.12701) (end 213.868 56.12701) (width 1) (layer F.Cu) (net 12))
   (segment (start 92.71 71.12) (end 95.25 68.58) (width 0.5) (layer F.Cu) (net 13))
   (segment (start 92.71 77.47) (end 92.71 71.12) (width 0.5) (layer F.Cu) (net 13) (status 10))
@@
   (segment (start 119.634 90.551) (end 117.120999 93.064001) (width 0.5) (layer B.Cu) (net 36) (status 10))
   (segment (start 117.120999 93.064001) (end 109.955001 93.064001) (width 0.5) (layer B.Cu) (net 36))
-  (segment (start 173.103999 79.276001) (end 173.103999 79.245001) (width 1) (layer F.Cu) (net 37))
-  (segment (start 171.834 80.546) (end 173.103999 79.276001) (width 1) (layer F.Cu) (net 37) (status 10))
-  (segment (start 173.103999 79.245001) (end 174.371 77.978) (width 1) (layer F.Cu) (net 37))
-  (segment (start 178.308 73.914) (end 173.99 78.232) (width 1) (layer F.Cu) (net 37))
-  (segment (start 178.308 73.914) (end 178.8795 73.3425) (width 1) (layer F.Cu) (net 37))
-  (segment (start 184.658 79.121) (end 186.563 79.121) (width 1) (layer F.Cu) (net 37))
-  (segment (start 178.8795 73.3425) (end 184.658 79.121) (width 1) (layer F.Cu) (net 37))
-  (segment (start 179.197 73.025) (end 178.8795 73.3425) (width 1) (layer F.Cu) (net 37))
-  (segment (start 179.197 62.23) (end 179.197 73.025) (width 1) (layer F.Cu) (net 37))
+  (segment (start 177.546 74.834) (end 177.546 59.817) (width 1) (layer F.Cu) (net 37) (status 20))
+  (segment (start 171.834 80.546) (end 177.546 74.834) (width 1) (layer F.Cu) (net 37) (status 10))
+  (segment (start 180.633001 77.921001) (end 177.546 74.834) (width 1) (layer F.Cu) (net 37))
+  (segment (start 185.363001 77.921001) (end 180.633001 77.921001) (width 1) (layer F.Cu) (net 37))
+  (segment (start 186.563 79.121) (end 185.363001 77.921001) (width 1) (layer F.Cu) (net 37) (status 10))
   (segment (start 96.393 75.184) (end 102.997 68.58) (width 0.5) (layer F.Cu) (net 38))
   (segment (start 102.997 68.58) (end 105.54863 68.58) (width 0.5) (layer F.Cu) (net 38))

Commit message: 0.2
Parts:
- moved GND6 0.76 mm to (81.7, 85.3)
- moved C11 0.51 mm to (88.1, 82.8)
- moved R9 0.51 mm to (93.2, 77.5)
- moved C6 0.51 mm to (88.8, 78.0)
Routing:
- net Net-(C11-Pad2): track 51.7 -> 50.7 mm
Changed lines of the file:
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@@
     (thickness 1.6)
     (drawings 11)
-    (tracks 325)
+    (tracks 323)
     (zones 0)
     (modules 77)
@@
   )
   (module Capacitor_THT:C_Rect_L7.0mm_W3.5mm_P5.00mm (layer F.Cu)
-    (at 87.63 82.804 270)
+    (at 88.138 82.804 270)
     (descr "C, Rect series, Radial, pin pitch=5.00mm, , length*width=7*3.5mm^2, Capacitor")
     (tags "C Rect series Radial pin pitch 5.00mm  length 7mm width 3.5mm Capacitor")
-    (fp_text reference C11 (at 2.413 -2.794 90) (layer F.SilkS)
+    (fp_text reference C11 (at 2.413 2.7305 90) (layer F.SilkS)
       (effects (font (size 1 1) (thickness 0.15)))
     )
@@
   )
   (module Capacitor_THT:C_Rect_L10.3mm_W5.0mm_P7.50mm_MKS4 (layer F.Cu)
-    (at 88.265 77.978 180)
+    (at 88.773 77.978 180)
     (descr "C, Rect series, Radial, pin pitch=7.50mm, , length*width=10.3*5mm^2, Capacitor, http://www.wima.com/EN/WIMA_MKS_4.pdf")
     (tags "C Rect series Radial pin pitch 7.50mm  length 10.3mm width 5mm Capacitor")
@@
   )
   (module Resistor_THT:R_Axial_DIN0207_L6.3mm_D2.5mm_P10.16mm_Horizontal (layer F.Cu)
-    (at 92.71 77.47 270)
+    (at 93.218 77.47 270)
     (descr "Resistor, Axial_DIN0207 series, Axial, Horizontal, pin pitch=10.16mm, 0.25W = 1/4W, length*diameter=6.3*2.5mm^2, http://cdn-reichelt.de/documents/datenblatt/B400/1_4W%23YAG.pdf")
     (tags "Resistor Axial_DIN0207 series Axial Horizontal pin pitch 10.16mm 0.25W = 1/4W length 6.3mm diameter 2.5mm")
@@
   )
   (module Connector_PinHeader_2.54mm:PinHeader_1x01_P2.54mm_Vertical (layer F.Cu)
-    (at 82.423 85.344)
+    (at 81.661 85.344)
     (descr "Through hole straight pin header, 1x01, 2.54mm pitch, single row")
     (tags "Through hole pin header THT 1x01 2.54mm single row")
@@
   (segment (start 91.44 107.188) (end 85.852 107.188) (width 0.5) (layer F.Cu) (net 9))
   (segment (start 85.852 107.188) (end 82.804 104.14) (width 0.5) (layer F.Cu) (net 9))
-  (segment (start 87.63 79.375) (end 87.63 82.55) (width 0.5) (layer F.Cu) (net 10) (status 20))
-  (segment (start 87.63 79.375) (end 89.027 77.978) (width 0.5) (layer F.Cu) (net 10) (status 20))
-  (segment (start 92.71 87.63) (end 87.63 82.804) (width 0.5) (layer B.Cu) (net 10) (status 30))
+  (segment (start 88.138 79.375) (end 88.138 82.55) (width 0.5) (layer F.Cu) (net 10) (status 20))
+  (segment (start 88.138 79.375) (end 89.535 77.978) (width 0.5) (layer F.Cu) (net 10) (status 20))
+  (segment (start 93.218 87.63) (end 88.138 82.804) (width 0.5) (layer B.Cu) (net 10) (status 30))
   (segment (start 65.405 68.58) (end 67.31 68.58) (width 0.5) (layer F.Cu) (net 11) (status 20))
   (segment (start 62.103 76.162) (end 62.103 71.882) (width 0.5) (layer F.Cu) (net 11) (status 10))
   (segment (start 62.103 71.882) (end 65.405 68.58) (width 0.5) (layer F.Cu) (net 11))
-  (segment (start 68.44137 68.58) (end 67.31 68.58) (width 0.5) (layer F.Cu) (net 11) (status 20))
-  (segment (start 72.781213 68.58) (end 68.44137 68.58) (width 0.5) (layer F.Cu) (net 11))
-  (segment (start 80.765 76.563787) (end 72.781213 68.58) (width 0.5) (layer F.Cu) (net 11))
-  (segment (start 80.765 77.978) (end 80.765 76.563787) (width 0.5) (layer F.Cu) (net 11) (status 10))
+  (segment (start 81.273 77.0185) (end 81.273 77.978) (width 0.5) (layer F.Cu) (net 11))
+  (segment (start 67.31 68.58) (end 72.8345 68.58) (width 0.5) (layer F.Cu) (net 11))
+  (segment (start 72.8345 68.58) (end 81.273 77.0185) (width 0.5) (layer F.Cu) (net 11))
   (segment (start 148.428 60.763) (end 151.419 63.754) (width 1) (layer F.Cu) (net 12))
   (segment (start 148.428 59.817) (end 148.428 60.763) (width 1) (layer F.Cu) (net 12) (status 10))
@@
   (segment (start 216.027 65.024) (end 216.027 58.166) (width 1) (layer F.Cu) (net 12))
   (segment (start 162.43999 56.12701) (end 213.868 56.12701) (width 1) (layer F.Cu) (net 12))
-  (segment (start 92.71 71.12) (end 95.25 68.58) (width 0.5) (layer F.Cu) (net 13))
-  (segment (start 92.71 77.47) (end 92.71 71.12) (width 0.5) (layer F.Cu) (net 13) (status 10))
-  (segment (start 95.25 68.58) (end 96.52 68.58) (width 0.5) (layer F.Cu) (net 13) (status 20))
-  (segment (start 92.71 82.47) (end 92.71 77.47) (width 0.5) (layer F.Cu) (net 13) (status 20))
-  (segment (start 92.416 82.764) (end 92.71 82.47) (width 0.5) (layer F.Cu) (net 13))
-  (segment (start 87.63 87.804) (end 92.416 82.764) (width 0.5) (layer F.Cu) (net 13) (status 10))
+  (segment (start 93.218 82.47) (end 93.218 77.47) (width 0.5) (layer F.Cu) (net 13) (status 20))
+  (segment (start 92.924 82.764) (end 93.218 82.47) (width 0.5) (layer F.Cu) (net 13))
+  (segment (start 88.138 87.804) (end 92.924 82.764) (width 0.5) (layer F.Cu) (net 13) (status 10))
   (segment (start 99.06 68.58) (end 96.52 68.58) (width 0.5) (layer B.Cu) (net 13) (status 20))
   (segment (start 104.267 72.39) (end 99.06 68.58) (width 0.5) (layer B.Cu) (net 13))
@@
   (segment (start 116.331 85.67) (end 114.245 85.67) (width 0.5) (layer B.Cu) (net 13) (status 10))
   (segment (start 114.245 85.67) (end 106.172 77.791733) (width 0.5) (layer B.Cu) (net 13))
+  (segment (start 93.218 71.882) (end 96.52 68.58) (width 0.5) (layer F.Cu) (net 13))
+  (segment (start 93.218 77.47) (end 93.218 71.882) (width 0.5) (layer F.Cu) (net 13))
   (segment (start 202.32263 104.394) (end 212.598 104.394) (width 1) (layer F.Cu) (net 14))
   (segment (start 198.501 99.441) (end 198.501 100.57237) (width 1) (layer F.Cu) (net 14) (status 10))

Commit message: BOM and other stuff.
Parts:
- removed B1: B1, Connector_PinHeader_2.54mm:PinHeader_1x01_P2.54mm_Vertical
- removed C17: 22n, Capacitor_THT:C_Rect_L10.3mm_W5.0mm_P7.50mm_MKS4
- removed PRESENCE1: PRESENCE, TerminalBlock_MetzConnect:TerminalBlock_MetzConnect_Type094_RT03502HBLU_1x02_P5.00mm_Horizontal
- AC1, BASS1, C1, C10, C11, C12, C13, C14, C15, C16, C2, C3, C4, C5, C6, C7, C8, C9, D1, D2, D3, D4, FIL1, G***, GAIN1, GND1, GND2, GND3, GND4, GND5, GND6, GND7, IN_HIGH_1, IN_LOW_1, LEVEL1, MID1, R1, R10, R11, R12, R13, R14, R15, R16, R17, R18, R19, R2, R21, R22, R23, R24, R25, R26, R3, R4, R5, R6, R7, R8, R9, Rbias1, TREBLE1: moved to B.Cu
- OUT1: footprint Connector_PinHeader_2.54mm:PinHeader_1x01_P2.54mm_Vertical -> TerminalBlock_MetzConnect:TerminalBlock_MetzConnect_Type094_RT03502HBLU_1x02_P5.00mm_Horizontal; moved to B.Cu
- moved IN_HIGH_1 16.2 mm to (66.0, 127.3), turned to 180 degrees
- moved IN_LOW_1 16.2 mm to (96.0, 127.3), turned to 180 degrees
- moved GAIN1 10.0 mm to (122.9, 128.5)
- moved BASS1 10.0 mm to (206.9, 128.5)
- moved LEVEL1 10.0 mm to (234.9, 128.5)
- moved TREBLE1 10.0 mm to (150.9, 128.5)
- moved MID1 9.99 mm to (178.9, 128.5)
- moved C12 6.99 mm to (225.0, 111.8)
- moved OUT1 5.08 mm to (148.5, 59.9), turned to 180 degrees
- moved C5 5.00 mm to (111.8, 105.3), turned to 90 degrees
- moved AC1 4.95 mm to (210.3, 59.9), turned to 180 degrees
- moved FIL1 4.95 mm to (170.2, 59.9), turned to 180 degrees
- moved GND4 4.95 mm to (197.5, 59.9), turned to 180 degrees
- moved G*** 0.85 mm to (125.9, 110.0), turned to 180 degrees
Connections:
- AC1 pad 1: /Tin2 -> /Tin1
- AC1 pad 2: /Tin1 -> /Tin2
- C5 pad 1: Net-(C4-Pad2) -> Net-(C5-Pad1)
- C5 pad 2: Net-(C5-Pad2) -> Net-(C4-Pad2)
- FIL1 pad 1: /FIL1 -> /FIL2
- FIL1 pad 2: /FIL2 -> /FIL1
- GAIN1 pad 2: Net-(C5-Pad2) -> Net-(C5-Pad1)
- OUT1 pad 1: /OUT -> /B1
- U1 pad 7: Net-(C5-Pad2) -> Net-(C5-Pad1)
Routing:
- net Net-(C5-Pad2): track 110.4 -> 0.00 mm
- net Net-(C5-Pad1): track 0.00 -> 110.3 mm
- net Net-(C17-Pad2): track 30.7 -> 0.00 mm
- net Net-(C1-Pad2): track 10.00 -> 32.4 mm
- net Net-(BASS1-Pad1): track 18.2 -> 39.6 mm
- net Net-(C4-Pad1): track 15.4 -> 28.2 mm
- net Net-(IN_HIGH_1-PadT): track 15.4 -> 27.3 mm
- net Net-(LEVEL1-Pad3): track 93.2 -> 83.4 mm
- net Net-(R2-Pad1): track 28.9 -> 19.2 mm
- net Net-(BASS1-Pad2): track 79.8 -> 73.0 mm, vias 0 -> 1
- net /B2: track 43.2 -> 49.6 mm
- net Net-(C4-Pad2): track 51.8 -> 51.1 mm, vias 0 -> 1
- net Net-(C14-Pad1): track 19.6 -> 18.9 mm
- net GND: track 0.00 -> 0.57 mm
Other:
- board text added: "Mount on the other side"
- board text added: "dazzmatazz@gmail.com"
- board text added: "v0.4"
- board text removed: "v0.2"
